File: lab1/amplifier/amplifier.kicad_pcb (KiCad board)
At the start: 2 copper layers, 44 x 40 mm, 29 parts, among them J1 Conn_Coaxial, J2 Conn_Coaxial, J3 Screw_Terminal_01x03, Q1 MMBT3904, Q2 MMBT3904, Q3 MMBT3906, Q4 MMBT3904, Q5 2N3904, Q6 2N3906

Commit message: Finish Lab 1
Parts:
- added C5: 1pF, Capacitor_SMD:C_0805_2012Metric, F.Cu at (72.0, 53.0)
- added C6: 0.1uF, Capacitor_SMD:C_0805_2012Metric, F.Cu at (67.0, 48.0)
- added C7: 0.1uF, Capacitor_SMD:C_0805_2012Metric, F.Cu at (67.0, 70.0)
- added C8: 10uF, Capacitor_SMD:C_0805_2012Metric, F.Cu at (67.0, 54.0)
- added C9: 10uF, Capacitor_SMD:C_0805_2012Metric, F.Cu at (60.0, 67.0)
- added R13: 24R, Resistor_SMD:R_0805_2012Metric, F.Cu at (87.0, 64.0)
- added R14: 24R, Resistor_SMD:R_0805_2012Metric, F.Cu at (89.0, 60.0)
- added R15: 24R, Resistor_SMD:R_0805_2012Metric, F.Cu at (87.0, 60.0)
- added R16: 24R, Resistor_SMD:R_0805_2012Metric, F.Cu at (89.0, 56.0)
- added R17: 24R, Resistor_SMD:R_0805_2012Metric, F.Cu at (87.0, 56.0)
- added R18: 24R, Resistor_SMD:R_0805_2012Metric, F.Cu at (89.0, 52.0)
- added R19: 24R, Resistor_SMD:R_0805_2012Metric, F.Cu at (87.0, 52.0)
- C3, C4, Q5, Q6: moved to B.Cu
- D1, D2: footprint Diode_SMD:D_SOD-123 -> Diode_THT:D_DO-35_SOD27_P7.62mm_Horizontal; moved to B.Cu
- R12: value 47R -> 24R
- moved C3 27.6 mm to (65.0, 47.0), turned to 270 degrees
- moved R3 16.4 mm to (72.0, 55.0)
- moved R12 10.8 mm to (89.0, 64.0), turned to 270 degrees
- moved J2 10.4 mm to (89.0, 48.0), turned to 90 degrees
- moved R4 10.4 mm to (69.0, 52.0), turned to 90 degrees
- moved R1 7.28 mm to (57.0, 54.0)
- moved Q4 7.00 mm to (68.0, 63.0), turned to 0 degrees
- moved R6 7.00 mm to (67.0, 67.0)
- moved Q1 6.32 mm to (56.0, 60.0)
- moved R10 4.23 mm to (82.4, 56.2)
- moved R2 4.12 mm to (56.0, 64.0), turned to 270 degrees
- moved R5 4.00 mm to (60.0, 54.0)
- moved Q6 3.42 mm to (78.4, 67.6)
- moved Q5 3.42 mm to (78.4, 56.6)
- moved R11 3.22 mm to (82.4, 62.2), turned to 180 degrees
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Connections:
- R12 pad 1: /SIG_OUT -> Net-(R12-Pad1)
Routing:
- net GND: track 2.10 -> 42.4 mm, vias 1 -> 4
- net Net-(D2-Pad1): track 35.1 -> 10.6 mm
- net Net-(C5-Pad2): track 37.5 -> 21.1 mm
- net +12V: track 76.0 -> 61.4 mm, vias 0 -> 2
- net Net-(Q5-Pad1): track 10.2 -> 3.23 mm
- net Net-(C2-Pad1): track 6.98 -> 12.8 mm
- net Net-(Q6-Pad1): track 11.8 -> 6.67 mm
- net Net-(D1-Pad1): track 7.70 -> 2.58 mm
- net Net-(C5-Pad1): track 33.7 -> 29.5 mm
- net Net-(D1-Pad2): track 20.5 -> 17.7 mm
- net Net-(Q2-Pad3): track 9.16 -> 11.5 mm
- net Net-(R17-Pad1): track 0.00 -> 2.12 mm
- net Net-(R16-Pad1): track 0.00 -> 2.12 mm
- net Net-(R15-Pad1): track 0.00 -> 2.12 mm
- net Net-(R14-Pad1): track 0.00 -> 2.12 mm
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Other:
- board text added: "Rev B"
- board text removed: "Rev A"
